Commit message: trajectory for bridge inspection

File: bluerov2_description/urdf/bridge3.urdf (robot description, URDF)
Before this commit: robot bridge2, 1 links, 0 joints
Links:
- removed link bridge2
- added link bridge3, mass 1456.8; collision mesh filename=package://bluerov2_description/meshes/bridge3.STL; visual mesh filename=package://bluerov2_description/meshes/bridge3.STL
