Commit message: init

File: bluerov2_description/urdf/base.xacro (robot description, xacro)
@@ -13,5 +13,5 @@
   -->
   <!-- Mass -->
-  <xacro:property name="mass" value="10"/>
+  <xacro:property name="mass" value="11.2"/>
   <!-- Describing the dimensions of the vehicle's bounding box: width, length, height -->
   <xacro:property name="x_size" value="0.448"/>
@@ -28,5 +28,5 @@
   assume NWU (otherwise cob is below cog?). 0.155
   -->
-  <xacro:property name="cob" value="0 0 0"/>
+  <xacro:property name="cob" value="0 0 0.3872"/>
   <!-- Fluid density -->
   <xacro:property name="rho" value="1028"/>
@@ -72,10 +72,10 @@
         </visual>
         <!-- In rexrov2_base they made collision planes to minize the GPU load -->
-        <!-- <collision>
+        <collision>
           <origin xyz="0 0 0" rpy="0 0 0"/>
           <geometry>
             <mesh filename="${collision_mesh_file}" scale="1 1 1" />
           </geometry>
-        </collision> -->
+        </collision>
       </link>
     <gazebo reference="${namespace}/base_link">

File: bluerov2_description/urdf/sensors.xacro (robot description, xacro)
@@ -17,11 +17,12 @@
     <origin xyz="0 0 0" rpy="0 0 0"/>
   </xacro:default_pressure>
-  <!-- Beacon Sensor  -->
-  <!-- <xacro:default_beacon namespace="${namespace}" parent_link="${namespace}/base_link">
-    <origin xyz="0 0 0" rpy="0 0 0"/>
-  </xacro:default_beacon> -->
   <!-- Mount a camera -->
-  <xacro:default_camera namespace="${namespace}" parent_link="${namespace}/base_link" suffix="">
-    <origin xyz="0.1 0 -0.2" rpy="0 0.6 0"/>
-  </xacro:default_camera>
+  <xacro:bluerov_camera namespace="" parent_link="${namespace}/base_link" suffix="_front">
+    <origin xyz="0.2 0 0" rpy="0 0 0"/>
+  </xacro:bluerov_camera>
+  <xacro:bluerov_camera namespace="" parent_link="${namespace}/base_link" suffix="_down">
+    <origin xyz="0 0 -0.2" rpy="0 ${pi/2} 0"/>
+  </xacro:bluerov_camera>
+  <!-- Mount a GPS. -->
+  <xacro:default_gps namespace="${namespace}" parent_link="${namespace}/base_link" />
 </robot>

File: bluerov2_description/urdf/snippets.xacro (robot description, xacro)
@@ -75,5 +75,5 @@
        <conversion>
          <type>Basic</type>
-         <rotorConstant>0.00001</rotorConstant>
+         <rotorConstant>0.0001</rotorConstant>
          <!-- <rotorConstant>0</rotorConstant> -->
        </conversion>
@@ -84,3 +84,134 @@
     </gazebo>
   </xacro:macro>
+  <xacro:macro name="bluerov_camera" params="namespace parent_link suffix *origin">
+    <xacro:regular_camera_plugin_macro
+      namespace="${namespace}"
+      suffix="${suffix}"
+      parent_link="${parent_link}"
+      topic="camera"
+      mass="0.001"
+      update_rate="30"
+      hfov="1.5125"
+      width="1920"
+      height="1080"
+      stddev="0.01"
+      scale="1.0">
+      <inertia ixx="0.00001" ixy="0.0" ixz="0.0" iyy="0.00001" iyz="0.0" izz="0.00001" />
+      <xacro:insert_block name="origin" />
+    </xacro:regular_camera_plugin_macro>
+  </xacro:macro>
+  <xacro:macro name="bluerov_altimeter"
+    params="namespace suffix parent_link *origin">
+    <!-- Sensor link -->
+    <link name="${namespace}/altimeter${suffix}_link">
+      <inertial>
+        <inertia ixx="0.00001" ixy="0.0" ixz="0.0" iyy="0.00001" iyz="0.0" izz="0.00001" />
+        <mass value="0.01" />
+        <origin xyz="0 0 0" rpy="0 0 0"/>
+      </inertial>
+      <visual>
+        <geometry>
+          <mesh filename="file://$(find bluerov2_description)/meshes/ping1d.dae" scale="1 1 1"/>
+        </geometry>
+        <origin xyz="0 0 0" rpy="0 0 -${0.5*pi}"/>
+      </visual>
+      <xacro:no_collision/>
+    </link>
+    <joint name="${namespace}_altimeter${suffix}_joint" type="revolute">
+      <xacro:insert_block name="origin" />
+      <parent link="${parent_link}" />
+      <child link="${namespace}/altimeter${suffix}_link" />
+      <limit upper="0" lower="0" effort="0" velocity="0" />
+      <axis xyz="1 0 0"/>
+    </joint>
+    <gazebo reference="${namespace}/altimeter${suffix}_link">
+      <sensor type="ray" name="sonar">
+          <pose>0 0 0 0 0 0</pose>
+          <update_rate>15.0</update_rate>
+          <ray>
+            <scan>
+              <horizontal>
+                <samples>5.0</samples>
+                <resolution>1</resolution>
+                <min_angle>-${15*pi/180}</min_angle>
+                <max_angle>${15*pi/180}</max_angle>
+              </horizontal>
+              <vertical>
+                <samples>5.0</samples>
+                <resolution>1</resolution>
+                <min_angle>-${15*pi/180}</min_angle>
+                <max_angle>${15*pi/180}</max_angle>
+              </vertical>
+            </scan>
+            <range>
+              <min>0.01</min>
+              <max>30.0</max>
+              <resolution>0.001</resolution>
+            </range>
+          </ray>
+          <plugin filename="libgazebo_ros_range.so" name="gazebo_ros_range">
+            <gaussianNoise>0.005</gaussianNoise>
+            <alwaysOn>true</alwaysOn>
+            <updateRate>15.0</updateRate>
+            <topicName>altimeter${suffix}</topicName>
+            <frameName>${namespace}/altimeter${suffix}_link</frameName>
+            <fov>${30*pi/180}</fov>
+            <radiation>ultrasound</radiation>
+          </plugin>
+        </sensor>
+    </gazebo>
+  </xacro:macro>
+  <xacro:macro name="bluerov2_sss"
+    params="namespace suffix parent_link topic mass update_rate
+      samples fov range_min range_max range_stddev mesh
+      *inertia *origin *visual">
+    <!-- Sensor link -->
+    <link name="${namespace}/sonar${suffix}_link">
+      <inertial>
+        <xacro:insert_block name="inertia" />
+        <mass value="${mass}" />
+        <origin xyz="0 0 0" rpy="0 0 0" />
+      </inertial>
+      <xacro:insert_block name="visual" />
+      <xacro:no_collision/>
+    </link>
+  <joint name="${namespace}_sonar${suffix}_joint" type="revolute">
+    <xacro:insert_block name="origin" />
+    <parent link="${parent_link}" />
+    <child link="${namespace}/sonar${suffix}_link" />
+    <limit upper="0" lower="0" effort="0" velocity="0" />
+    <axis xyz="1 0 0"/>
+  </joint>
+  <gazebo reference="${namespace}/sonar${suffix}_link">
+    <sensor type="ray" name="sonar${suffix}">
+      <pose>0 0 0 0 0 0</pose>
+      <visualize>true</visualize>
+      <update_rate>${update_rate}</update_rate>
+      <ray>
+        <scan>
+          <horizontal>
+            <samples>${samples}</samples>
+            <resolution>1</resolution>
+            <min_angle>-${0.5*fov}</min_angle>
+            <max_angle>${0.5*fov}</max_angle>
+          </horizontal>
+        </scan>
+        <range>
+          <min>${range_min}</min>
+          <max>${range_max}</max>
+          <resolution>0.01</resolution>
+        </range>
+        <noise>
+          <type>gaussian</type>
+          <mean>0.0</mean>
+          <stddev>${range_stddev}</stddev>
+        </noise>
+      </ray>
+      <plugin name="sonar${suffix}_controller" filename="libgazebo_ros_laser.so">
+        <topicName>${topic}${suffix}</topicName>
+        <frameName>sonar${suffix}_link</frameName>
+      </plugin>
+    </sensor>
+  </gazebo>
+  </xacro:macro>
 </robot>

Commit message: May 16 Stage changes before solving some issue

File: bluerov2_description/urdf/base.xacro (robot description, xacro)
@@ -78,4 +78,19 @@
           </geometry>
         </collision>
+        <!-- <light name="light_source1" type="spot">
+          <pose frame=''>0.25 0 0.25 0 -0.7854 0</pose>
+          <attenuation>
+            <range>30</range>
+            <linear>0.05</linear>
+          </attenuation>
+          <diffuse>1 0 0 1</diffuse>
+          <specular>1 0 0 1</specular>
+          <spot>
+            <inner_angle>0.3</inner_angle>
+            <outer_angle>0.35</outer_angle>
+            <falloff>1</falloff>
+          </spot>
+          <direction>0 0 -1</direction>
+        </light> -->
       </link>
     <gazebo reference="${namespace}/base_link">

File: bluerov2_description/urdf/sensors.xacro (robot description, xacro)
@@ -25,7 +25,11 @@
   </xacro:bluerov_camera> -->
   <!-- Mount a DVL -->
-  <xacro:default_dvl namespace="${namespace}" parent_link="${namespace}/base_link">
-    <origin xyz="0 0 -0.2" rpy="0 -1.5708 0"/>
-  </xacro:default_dvl>
+  <!-- <xacro:include filename="$(find teledyne_whn_uuvsim_description)/urdf/teledyne_whn.xacro"/>
+  <xacro:teledyne_whn_enu_macro namespace="${namespace}" parent_link="${namespace}/base_link">
+    <origin xyz="0 0 -0.2" rpy="0 ${0.5*pi} 0"/>
+  </xacro:teledyne_whn_enu_macro> -->
+  <!-- <xacro:default_dvl namespace="${namespace}" parent_link="${namespace}/base_link">
+    <origin xyz="0 0 -0.2" rpy="0 ${0.5*pi} 0"/>
+  </xacro:default_dvl> -->
   <!-- Mount a GPS. -->
   <xacro:default_gps namespace="${namespace}" parent_link="${namespace}/base_link" />
