Commit message: mount stereo camera

File: bluerov2_description/urdf/sensors.xacro (robot description, xacro)
@@ -18,11 +18,19 @@
   </xacro:default_pressure>
   <!-- Mount a camera -->
-  <xacro:bluerov_camera namespace="" parent_link="${namespace}/base_link" suffix="_front">
+  <!-- <xacro:bluerov_camera namespace="" parent_link="${namespace}/base_link" suffix="_front">
     <origin xyz="0.2 0 0" rpy="0 0 0"/>
-  </xacro:bluerov_camera>
-  <xacro:bluerov_camera namespace="" parent_link="${namespace}/base_link" suffix="_down">
+  </xacro:bluerov_camera> -->
+  <!-- <xacro:bluerov_camera namespace="" parent_link="${namespace}/base_link" suffix="_down">
     <origin xyz="0 0 -0.2" rpy="0 ${pi/2} 0"/>
-  </xacro:bluerov_camera>
+  </xacro:bluerov_camera> -->
   <!-- Mount a GPS. -->
   <xacro:default_gps namespace="${namespace}" parent_link="${namespace}/base_link" />
+  <!-- Mount a stereo camera -->
+  <!-- <xacro:include filename="$(find bluerov2_description)/urdf/_d435.urdf.xacro" />
+  <sensor_d435 parent="${namespace}/base_link">
+  </sensor_d435> -->
+  <xacro:include filename="$(find bluerov2_description)/urdf/_d435.urdf.xacro" />
+  <sensor_d435 parent="${namespace}/base_link">
+    <origin xyz="0.2 0 0" rpy="0 0 0"/>
+  </sensor_d435>
 </robot>

Commit message: New swimming pool scenario (side), Add DVL

File: bluerov2_description/urdf/sensors.xacro (robot description, xacro)
@@ -24,5 +24,12 @@
     <origin xyz="0 0 -0.2" rpy="0 ${pi/2} 0"/>
   </xacro:bluerov_camera> -->
+  <!-- Mount a DVL -->
+  <xacro:default_dvl namespace="${namespace}" parent_link="${namespace}/base_link">
+    <origin xyz="0 0 -0.2" rpy="0 -1.5708 0"/>
+  </xacro:default_dvl>
   <!-- Mount a GPS. -->
   <xacro:default_gps namespace="${namespace}" parent_link="${namespace}/base_link" />
+  <!-- Mount a light -->
+  <!-- <xacro:include filename="$(find uuv_sensor_ros_plugins)/urdf/light.xacro"/>
+    <xacro:point_light namespace="${namespace}" parent_link="${namespace}/base_link"/> -->
 </robot>

Commit message: update a bit after adding dvl sub

File: bluerov2_description/urdf/sensors.xacro (robot description, xacro)
@@ -29,7 +29,11 @@
     <origin xyz="0 0 -0.2" rpy="0 ${0.5*pi} 0"/>
   </xacro:teledyne_whn_enu_macro> -->
-  <!-- <xacro:default_dvl namespace="${namespace}" parent_link="${namespace}/base_link">
+  <xacro:default_dvl namespace="${namespace}" parent_link="${namespace}/base_link">
     <origin xyz="0 0 -0.2" rpy="0 ${0.5*pi} 0"/>
-  </xacro:default_dvl> -->
+  </xacro:default_dvl>
+  <!-- Mount a sonar -->
+  <xacro:forward_multibeam_p900 namespace="${namespace}" parent_link="${namespace}/base_link">
+    <origin xyz="0 0 -0.2" rpy="0 0 0"/>
+  </xacro:forward_multibeam_p900>
   <!-- Mount a GPS. -->
   <xacro:default_gps namespace="${namespace}" parent_link="${namespace}/base_link" />

Commit message: Update pool_traj, Use sensor fusion estimates

File: bluerov2_description/urdf/sensors.xacro (robot description, xacro)
@@ -10,7 +10,10 @@
   <xacro:default_pose_3d namespace="${namespace}" parent_link="${namespace}/base_link" />
   <!-- IMU Sensor -->
-  <xacro:default_imu namespace="${namespace}" parent_link="${namespace}/base_link">
+  <!-- <xacro:default_imu namespace="${namespace}" parent_link="${namespace}/base_link">
     <origin xyz="0 0 0" rpy="0 0 0"/>
-  </xacro:default_imu>
+  </xacro:default_imu> -->
+    <xacro:default_imu_svin namespace="${namespace}" parent_link="${namespace}/base_link">
+    <origin xyz="0 0 0" rpy="0 0 0"/>
+  </xacro:default_imu_svin>
   <!-- Pressure Sensor  -->
   <xacro:default_pressure namespace="${namespace}" parent_link="${namespace}/base_link">
@@ -30,5 +33,6 @@
   </xacro:teledyne_whn_enu_macro> -->
   <xacro:default_dvl namespace="${namespace}" parent_link="${namespace}/base_link">
-    <origin xyz="0 0 -0.2" rpy="0 ${0.5*pi} 0"/>
+    <!-- <origin xyz="0 0 -0.2" rpy="0 ${0.5*pi} 0"/> -->
+    <origin xyz="0 0 -0.2" rpy="0 0 0"/>
   </xacro:default_dvl>
   <!-- Mount a sonar -->
@@ -38,4 +42,9 @@
   <!-- Mount a GPS. -->
   <xacro:default_gps namespace="${namespace}" parent_link="${namespace}/base_link" />
+  <!-- Mount a stereo camera -->
+  <xacro:include filename="$(find uuv_sensor_ros_plugins)/urdf/stereo_snippets.xacro"/>
+  <xacro:duo3d_camera namespace="${namespace}" parent_link="${namespace}/base_link">
+    <origin xyz="0.2 0 0" rpy="0 0 0"/>
+  </xacro:duo3d_camera>
   <!-- Mount a light -->
   <!-- <xacro:include filename="$(find uuv_sensor_ros_plugins)/urdf/light.xacro"/>
